File: Benjolin Panel.kicad_pcb (KiCad board)
At the start: 2 copper layers, 80.1 x 128.7 mm, 60 parts

Commit message: Update panel files
Parts:
- removed the G*** at (96.5, 127.0)
- removed the G*** at (75.3, 80.2)
- removed the G*** at (75.3, 56.1)
- removed the G*** at (86.9, 34.4)
- removed the G*** at (52.7, 125.3)
- removed the G*** at (52.8, 101.3)
- removed the G*** at (52.8, 77.7)
- removed the G*** at (52.8, 53.8)
- removed the G*** at (75.3, 127.0)
- removed the G*** at (119.2, 103.5)
- removed the G*** at (96.5, 103.6)
- removed the G*** at (119.2, 80.0)
- removed the G*** at (119.2, 56.0)
- removed the G*** at (96.5, 80.1)
- removed the G*** at (96.5, 56.1)
- removed the G*** at (75.3, 103.6)
- removed the ~ at (86.9, 151.6)
- removed the ~ at (109.2, 123.4)
- removed the ~ at (109.2, 111.4)
Other:
- board text added: "BENJOLIN"
- board text added: "CV A"
- board text added: "CV B"
- board text added: "CV F"
- board text added: "EMPHASIS"
- board text added: "EXT"
- board text added: "FREQ"
- board text added: "FREQ A"
- board text added: "FREQ B"
- board text added: "FREQ CV"
- board text added: "JLCJLCJLCJLC"
- board text added: "LOOP OFFSET"
- board text added: "OFF"
- board text added: "ON"
- board text added: "RUNGLER B"
- board text added: "RUNGLER CV"
- board text added: "RUNGLER FILTER"
